File: Lobotomizer_Fuzz.sch (KiCad schematic (older format))
At the start: 77 parts, among them Q1 NTE467, Q2 2N5089, Q3 2N5087, Q4 2N5089, Q5 NTE467, Q6 BS170, SW1 SW_SPDT_MSM, SW2 SW_SPDT, SW3 SW_SPDT, U1 LM741

Commit message: lobotomizer v2 update
so much changed i cant note it all here
Parts:
- removed C1, C11, C18: 100p, Capacitor_THT:C_Disc_D4.7mm_W2.5mm_P5.00mm, symbol Device:C
- removed C10: 30p, Capacitor_THT:C_Rect_L4.0mm_W2.5mm_P2.50mm, symbol Device:C
- removed C12: 2.2p, Capacitor_THT:C_Rect_L4.0mm_W2.5mm_P2.50mm, symbol Device:C
- removed C13, C14: 4.7u, Capacitor_THT:CP_Radial_D5.0mm_P2.00mm, symbol Device:C
- removed C15: 3.3n, Capacitor_THT:C_Rect_L4.0mm_W2.5mm_P2.50mm, symbol Device:C
- removed C16, C8: 22n, Capacitor_THT:C_Disc_D4.3mm_W1.9mm_P5.00mm, symbol Device:C
- removed C17, C19, C3, C7: 1u, Capacitor_THT:CP_Radial_D5.0mm_P2.00mm, symbol Device:C
- removed C2, C22, C4, C5, C6: 100n, Capacitor_THT:C_Disc_D3.8mm_W2.6mm_P2.50mm, symbol Device:C
- removed C20, C23: 10u, Capacitor_THT:CP_Radial_D5.0mm_P2.00mm, symbol Device:C
- removed C21: 100u, Capacitor_THT:CP_Radial_D5.0mm_P2.00mm, symbol Device:CP
- removed C9: 1n, Capacitor_THT:C_Disc_D5.0mm_W2.5mm_P2.50mm, symbol Device:C
- removed D1, D2, D3, D5, D6, D7: 4148, Diode_THT:D_DO-35_SOD27_P7.62mm_Horizontal, symbol Device:D
- removed D4: LED, LED_THT:LED_D5.0mm, symbol Device:LED
- removed D8: 5817, Diode_THT:D_DO-41_SOD81_P7.62mm_Horizontal, symbol Device:D
- removed Q1, Q5: NTE467, Package_TO_SOT_THT:TO-92_Inline, symbol Device:Q_NJFET_DSG
- removed Q2, Q4: 2N5089, Package_TO_SOT_THT:TO-92_Inline, symbol Device:Q_NPN_EBC
- removed Q3: 2N5087, Package_TO_SOT_THT:TO-92_Inline, symbol Device:Q_PNP_EBC
- removed Q6: BS170, Package_TO_SOT_THT:TO-92_Inline, symbol Transistor_FET:BS170
- removed R1, R16, R22, R24, R3: 1M, Resistor_THT:R_Axial_DIN0207_L6.3mm_D2.5mm_P7.62mm_Horizontal, symbol Device:R
- removed R10, R15, R23, R28, R30, R31, R9: 10K, Resistor_THT:R_Axial_DIN0207_L6.3mm_D2.5mm_P7.62mm_Horizontal, symbol Device:R
- removed R11, R12: 100K, Resistor_THT:R_Axial_DIN0207_L6.3mm_D2.5mm_P10.16mm_Horizontal, symbol Device:R
- removed R13, R14, R6: 47K, Resistor_THT:R_Axial_DIN0207_L6.3mm_D2.5mm_P7.62mm_Horizontal, symbol Device:R
- removed R17, R2, R20, R25, R4: 1K, Resistor_THT:R_Axial_DIN0207_L6.3mm_D2.5mm_P7.62mm_Horizontal, symbol Device:R
- removed R18: 47, Resistor_THT:R_Axial_DIN0207_L6.3mm_D2.5mm_P7.62mm_Horizontal, symbol Device:R
- removed R19: 560, Resistor_THT:R_Axial_DIN0207_L6.3mm_D2.5mm_P7.62mm_Horizontal, symbol Device:R
- removed R21: 1.5K, Resistor_THT:R_Axial_DIN0207_L6.3mm_D2.5mm_P7.62mm_Horizontal, symbol Device:R
- removed R26, R27, R5: 470K, Resistor_THT:R_Axial_DIN0207_L6.3mm_D2.5mm_P7.62mm_Horizontal, symbol Device:R
- removed R29: 470, Resistor_THT:R_Axial_DIN0204_L3.6mm_D1.6mm_P5.08mm_Horizontal, symbol Device:R
- removed R7: 22K, Resistor_THT:R_Axial_DIN0207_L6.3mm_D2.5mm_P7.62mm_Horizontal, symbol Device:R
- removed R8: 2.2K, Resistor_THT:R_Axial_DIN0207_L6.3mm_D2.5mm_P7.62mm_Horizontal, symbol Device:R
- removed RV1: 50K, Potentiometer_THT:Potentiometer_Bourns_3266Y_Vertical, symbol Device:R_POT
- removed RV2, RV3, RV4, RV5: 100K, Potentiometer_THT:Potentiometer_Bourns_3266Y_Vertical, symbol Device:R_POT
- removed SW1: SW_SPDT_MSM, Button_Switch_THT:SW_Slide_1P2T_CK_OS102011MS2Q, symbol Switch:SW_SPDT_MSM
- removed SW2, SW3: SW_SPDT, Button_Switch_THT:SW_Slide_1P2T_CK_OS102011MS2Q, symbol Switch:SW_SPDT
- removed U1: LM741, Package_DIP:DIP-8_W7.62mm, symbol Amplifier_Operational:LM741
- added C101, C106: 100n, Capacitor_THT:C_Disc_D3.8mm_W2.6mm_P2.50mm, symbol Device:C
- added C102: 10n, Capacitor_THT:C_Disc_D4.3mm_W1.9mm_P5.00mm, symbol Device:C
- added C103: 470p, Capacitor_THT:C_Disc_D4.3mm_W1.9mm_P5.00mm, symbol Device:C
- added C104, C105: 4.7u, Capacitor_THT:CP_Radial_D5.0mm_P2.00mm, symbol Device:CP
- added C107: 330n, Capacitor_THT:CP_Radial_D5.0mm_P2.00mm, symbol Device:C
- added Q101, Q102: 5089, Package_TO_SOT_THT:TO-92_Inline, symbol Device:Q_NPN_EBC
- added Q103: 5308, Package_TO_SOT_THT:TO-92_Inline, symbol Device:Q_NPN_Darlington_EBC
- added R101, R103, R108: 910K, Resistor_THT:R_Axial_DIN0207_L6.3mm_D2.5mm_P7.62mm_Horizontal, symbol Device:R
- added R102, R106: 180K, Resistor_THT:R_Axial_DIN0207_L6.3mm_D2.5mm_P7.62mm_Horizontal, symbol Device:R
- added R104: 910, Resistor_THT:R_Axial_DIN0207_L6.3mm_D2.5mm_P7.62mm_Horizontal, symbol Device:R
- added R105: 10K, Resistor_THT:R_Axial_DIN0207_L6.3mm_D2.5mm_P7.62mm_Horizontal, symbol Device:R
- added R107: 4.7M, Resistor_THT:R_Axial_DIN0207_L6.3mm_D2.5mm_P10.16mm_Horizontal, symbol Device:R
- added R109: 750, Resistor_THT:R_Axial_DIN0204_L3.6mm_D1.6mm_P5.08mm_Horizontal, symbol Device:R
- added RV101, RV105: 100K, Potentiometer_THT:Potentiometer_Bourns_3266Y_Vertical, symbol Device:R_POT
- added RV102: 50K, Potentiometer_THT:Potentiometer_Bourns_3266Y_Vertical, symbol Device:R_POT
- added RV103, RV104: 10K, Potentiometer_THT:Potentiometer_Bourns_3266Y_Vertical, symbol Device:R_POT
- added SW101: SW_SPDT_MSM, TerminalBlock_Phoenix:TerminalBlock_Phoenix_MKDS-1,5-3-5.08_1x03_P5.08mm_Horizontal, symbol Switch:SW_SPDT_MSM
Connections:
- net FUZZ_OUT: now also RV105.3
- net GND: now also C107.2, R104.2, R108.2, RV103.1, RV105.1, SW101.2
- net VCLEAN: now also R101.1, R102.1, R103.1, R106.1, R107.1, RV102.3
- new net: C101.1, RV101.3
- new net: C102.1, C103.2, Q101.2 (B), R101.2, RV101.1, RV101.2
- new net: Q101.1 (E), SW101.1
- new net: C103.1, C104.1, Q101.3 (C), R102.2
- new net: C104.2, Q102.2 (B), R103.2, R104.1
- new net: R105.1, SW101.3
- new net: Q102.1 (E), R105.2
- new net: C105.1, Q102.3 (C), R106.2
- new net: C105.2, Q103.2 (B), R107.2, R108.1
- new net: Q103.1 (E), RV103.2
- new net: C106.2, Q103.3 (C), R109.2
- new net: R109.1, RV102.1, RV102.2
- new net: C106.1, RV104.2, RV104.3, RV105.2
- new net: C107.1, RV104.1
- new net SIGNAL_IN: C101.2, C102.2
- no-connect marks 0 -> 1
Other:
- note removed: "BOOST SELECT\n"
- note removed: "BOOST!!\n"
- note removed: "CLIPPING"
- note removed: "DISTORTION\n"
- note removed: "FILTER"
- note removed: "FX_OUT"
- note removed: "OCTAVE"
- note removed: "POWER"
- note removed: "VOLUME\n"
