File: Lobotomizer_Saw.sch (KiCad schematic (older format))
At the start: 37 parts, among them Q201 MPSA05, Q202 MPSA05, SW201 SW_SPDT, SW202 SW_SPDT, U201 LM386, U202 TL072

Commit message: finalized v1 design
Changed lines of the file:
@@
 Wire Wire Line
 	3300 2800 2850 2800
-Wire Wire Line
-	2550 2800 2550 3000
-Text HLabel 2550 3000 3    50   Output Italic 10
-BYPASS_KILL
 Connection ~ 2850 2800
 Wire Wire Line
@@
 Text GLabel 8750 5650 0    50   Output Italic 10
 SIGNAL_OUT
-Text HLabel 9500 4800 0    50   Input Italic 10
-BYPASS_KILL
 $Comp
 L power:+9V #PWR0143
@@
 Text Notes 2350 5850 0    70   Italic 14
 POWER\n
+Wire Wire Line
+	2550 4800 9500 4800
+Wire Wire Line
+	2550 2800 2550 4800
 $EndSCHEMATC

Commit message: lobotomizer v2 update
so much changed i cant note it all here
Parts:
- removed C209: 100n, Capacitor_THT:C_Disc_D3.8mm_W2.6mm_P2.50mm, symbol Device:C
- removed R208, R209, R210, R211: 100K, Resistor_THT:R_Axial_DIN0207_L6.3mm_D2.5mm_P10.16mm_Horizontal, symbol Device:R
- removed RV203, RV204, RV205: 100K, Potentiometer_THT:Potentiometer_Bourns_3266Y_Vertical, symbol Device:R_POT
- removed SW201, SW202: SW_SPDT, Button_Switch_THT:SW_Slide_1P2T_CK_OS102011MS2Q, symbol Switch:SW_SPDT
- removed U202: TL072, Package_DIP:DIP-8_W7.62mm, symbol Amplifier_Operational:TL072
- added SW301: SW_SPDT, TerminalBlock_Phoenix:TerminalBlock_Phoenix_MKDS-1,5-3-5.08_1x03_P5.08mm_Horizontal, symbol Switch:SW_SPDT
- R305: renamed from R205; footprint Resistor_THT:R_Axial_DIN0207_L6.3mm_D2.5mm_P7.62mm_Horizontal -> Resistor_THT:R_Axial_DIN0204_L3.6mm_D1.6mm_P5.08mm_Horizontal
- R306: renamed from R206; footprint Resistor_THT:R_Axial_DIN0207_L6.3mm_D2.5mm_P7.62mm_Horizontal -> Resistor_THT:R_Axial_DIN0204_L3.6mm_D1.6mm_P5.08mm_Horizontal
- renumbered C201 to C301, C202 to C302, C203 to C303, C204 to C304, C205 to C305, C206 to C306, C207 to C307, C208 to C308, D201 to D301, D202 to D302, D203 to D303, D204 to D304, D205 to D305, D206 to D306, Q201 to Q301, Q202 to Q302, R201 to R301, R202 to R302, R203 to R303, R204 to R304, R207 to R307, RV201 to RV301, RV202 to RV302, U201 to U301
Connections:
- net SAW_OUT: now reaches D303.2 (A), D304.1 (K), R306.1
- net REVERB_OUT: no longer names the net of C301.2
- net REVERB_OUT: now also SW301.2 (B)
- new net MEGAFUCKER_OUT: SW301.1 (A)
- new net SIGNAL_IN: SW301.3 (C)
Other:
- note removed: "DEATH METER"
